Commit message: my_cafe.world add

File: project_ws/src/uner_bot/urdf/UNER_bot.xacro (robot description, xacro)
@@ -16,5 +16,5 @@
   <link name="robot_footprint"></link>
   <joint name="robot_footprint_joint" type="fixed">
-    <origin xyz="0 0 0" rpy="0 0 0" />
+    <origin xyz="0 0 0.1" rpy="0 0 0" />
     <parent link="robot_footprint"/>
     <child link="chassis" />
